File: v1/Joysticks.kicad_sch (KiCad schematic)
At the start: 9 parts, among them J11 DB9_Male_MountingHoles, J12 DB9_Male_MountingHoles, J13 Conn_02x06_Odd_Even, U4 74LV165A, U5 74LV165A

Commit message: Updated VGA jumper block from 3x6 to 3x8
Parts:
- renumbered J11 to J10, J12 to J11, J13 to J12
Changed lines of the file:
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@@
   (symbol (lib_id "Connector_Generic:Conn_02x06_Odd_Even") (at 62.23 176.53 0) (mirror x) (unit 1)
     (in_bom yes) (on_board yes) (fields_autoplaced)
-    (property "Reference" "J13" (id 0) (at 63.5 162.56 0))
+    (property "Reference" "J12" (id 0) (at 63.5 162.56 0))
     (property "Value" "Conn_02x06_Odd_Even" (id 1) (at 63.5 165.1 0))
     (property "Footprint" "Connector_PinHeader_2.54mm:PinHeader_2x06_P2.54mm_Vertical" (id 2) (at 62.23 176.53 0)
@@
   (symbol (lib_id "Connector:DB9_Male_MountingHoles") (at 60.96 52.07 180) (unit 1)
     (in_bom yes) (on_board yes)
-    (property "Reference" "J11" (id 0) (at 62.23 66.04 0)
+    (property "Reference" "J10" (id 0) (at 62.23 66.04 0)
       (effects (font (size 1.27 1.27)) (justify left))
     )
@@
   (symbol (lib_id "Connector:DB9_Male_MountingHoles") (at 60.96 116.84 180) (unit 1)
     (in_bom yes) (on_board yes)
-    (property "Reference" "J12" (id 0) (at 62.23 130.81 0)
+    (property "Reference" "J11" (id 0) (at 62.23 130.81 0)
       (effects (font (size 1.27 1.27)) (justify left))
     )

Commit message: Silk screen
Parts:
- renumbered J12 to JP5
Changed lines of the file:
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@@
   (symbol (lib_id "Connector_Generic:Conn_02x06_Odd_Even") (at 62.23 176.53 0) (mirror x) (unit 1)
     (in_bom yes) (on_board yes) (fields_autoplaced)
-    (property "Reference" "J12" (id 0) (at 63.5 162.56 0))
+    (property "Reference" "JP5" (id 0) (at 63.5 162.56 0))
     (property "Value" "Conn_02x06_Odd_Even" (id 1) (at 63.5 165.1 0))
     (property "Footprint" "Connector_PinHeader_2.54mm:PinHeader_2x06_P2.54mm_Vertical" (id 2) (at 62.23 176.53 0)

Commit message: Added jumpers for Pi and Joystick power
Parts:
- added JP7, JP8: Jumper_2_Open, Connector_PinHeader_2.54mm:PinHeader_1x02_P2.54mm_Vertical, symbol Jumper:Jumper_2_Open
Connections:
- net +5V: now also JP7.1 (A), JP8.1 (A); no longer J10.7, J11.7
- new net: J10.7, JP8.2 (B)
- new net: J11.7, JP7.2 (B)
Changed lines of the file:
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@@
     (pin "9")
+  )
+  (symbol (lib_id "Jumper:Jumper_2_Open") (at 71.12 30.48 270) (unit 1)
+    (in_bom yes) (on_board yes) (fields_autoplaced)
+    (property "Reference" "JP8" (id 0) (at 73.66 29.2099 90)
+      (effects (font (size 1.27 1.27)) (justify left))
+    )
+    (property "Value" "Jumper_2_Open" (id 1) (at 73.66 31.7499 90)
+      (effects (font (size 1.27 1.27)) (justify left))
+    )
+    (property "Footprint" "Connector_PinHeader_2.54mm:PinHeader_1x02_P2.54mm_Vertical" (id 2) (at 71.12 30.48 0)
+      (effects (font (size 1.27 1.27)) hide)
+    )
+    (property "Datasheet" "~" (id 3) (at 71.12 30.48 0)
+      (effects (font (size 1.27 1.27)) hide)
+    )
+    (pin "1")
+    (pin "2")
   )
   (symbol (lib_id "power:GND") (at 151.13 72.39 0) (unit 1)
@@
     (pin "1")
   )
-  (symbol (lib_id "power:+5V") (at 71.12 35.56 0) (unit 1)
-    (in_bom yes) (on_board yes) (fields_autoplaced)
-    (property "Reference" "#PWR040" (id 0) (at 71.12 39.37 0)
-      (effects (font (size 1.27 1.27)) hide)
-    )
-    (property "Value" "+5V" (id 1) (at 71.12 30.48 0))
-    (property "Footprint" "" (id 2) (at 71.12 35.56 0)
-      (effects (font (size 1.27 1.27)) hide)
-    )
-    (property "Datasheet" "" (id 3) (at 71.12 35.56 0)
+  (symbol (lib_id "power:+5V") (at 71.12 25.4 0) (unit 1)
+    (in_bom yes) (on_board yes) (fields_autoplaced)
+    (property "Reference" "#PWR040" (id 0) (at 71.12 29.21 0)
+      (effects (font (size 1.27 1.27)) hide)
+    )
+    (property "Value" "+5V" (id 1) (at 71.12 20.32 0))
+    (property "Footprint" "" (id 2) (at 71.12 25.4 0)
+      (effects (font (size 1.27 1.27)) hide)
+    )
+    (property "Datasheet" "" (id 3) (at 71.12 25.4 0)
       (effects (font (size 1.27 1.27)) hide)
     )
@@
     (pin "9")
   )
+  (symbol (lib_id "Jumper:Jumper_2_Open") (at 71.12 95.25 270) (unit 1)
+    (in_bom yes) (on_board yes) (fields_autoplaced)
+    (property "Reference" "JP7" (id 0) (at 73.66 93.9799 90)
+      (effects (font (size 1.27 1.27)) (justify left))
+    )
+    (property "Value" "Jumper_2_Open" (id 1) (at 73.66 96.5199 90)
+      (effects (font (size 1.27 1.27)) (justify left))
+    )
+    (property "Footprint" "Connector_PinHeader_2.54mm:PinHeader_1x02_P2.54mm_Vertical" (id 2) (at 71.12 95.25 0)
+      (effects (font (size 1.27 1.27)) hide)
+    )
+    (property "Datasheet" "~" (id 3) (at 71.12 95.25 0)
+      (effects (font (size 1.27 1.27)) hide)
+    )
+    (pin "1")
+    (pin "2")
+  )
   (symbol (lib_id "power:GND") (at 71.12 130.81 0) (unit 1)
     (in_bom yes) (on_board yes) (fields_autoplaced)
@@
     (pin "1")
   )
-  (symbol (lib_id "power:+5V") (at 71.12 100.33 0) (unit 1)
-    (in_bom yes) (on_board yes) (fields_autoplaced)
-    (property "Reference" "#PWR042" (id 0) (at 71.12 104.14 0)
-      (effects (font (size 1.27 1.27)) hide)
-    )
-    (property "Value" "+5V" (id 1) (at 71.12 95.25 0))
-    (property "Footprint" "" (id 2) (at 71.12 100.33 0)
-      (effects (font (size 1.27 1.27)) hide)
-    )
-    (property "Datasheet" "" (id 3) (at 71.12 100.33 0)
-      (effects (font (size 1.27 1.27)) hide)
-    )
+  (symbol (lib_id "power:+5V") (at 71.12 90.17 0) (unit 1)
+    (in_bom yes) (on_board yes) (fields_autoplaced)
+    (property "Reference" "#PWR042" (id 0) (at 71.12 93.98 0)
+      (effects (font (size 1.27 1.27)) hide)
+    )
+    (property "Value" "+5V" (id 1) (at 71.12 85.09 0))
+    (property "Footprint" "" (id 2) (at 71.12 90.17 0)
+      (effects (font (size 1.27 1.27)) hide)
+    )
+    (property "Datasheet" "" (id 3) (at 71.12 90.17 0)
+      (effects (font (size 1.27 1.27)) hide)
+    )

Commit message: Tidy around Joystick connectors
Connections:
- net Cfg0: now also RN2.7 (R6); no longer RN2.4 (R3)
- net Cfg1: now also RN2.8 (R7); no longer RN2.3 (R2)
- net Cfg2: now also RN2.9 (R8); no longer RN2.2 (R1)
- net JS1_Down: now also RN2.3 (R2); no longer RN2.8 (R7)
- net JS1_Fire: now also RN2.6 (R5); no longer RN2.5 (R4)
- net JS1_Left: now also RN2.4 (R3); no longer RN2.7 (R6)
- net JS1_Right: now also RN2.5 (R4); no longer RN2.6 (R5)
- net JS1_Up: now also RN2.2 (R1); no longer RN2.9 (R8)
Changed lines of the file:
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@@
     (pin "1")
   )
-  (symbol (lib_id "Device:R_Network08") (at 118.11 92.71 0) (unit 1)
-    (in_bom yes) (on_board yes) (fields_autoplaced)
-    (property "Reference" "RN2" (id 0) (at 128.27 91.6939 0)
+  (symbol (lib_id "Device:R_Network08") (at 115.57 92.71 0) (mirror y) (unit 1)
+    (in_bom yes) (on_board yes)
+    (property "Reference" "RN2" (id 0) (at 132.08 92.71 0)
       (effects (font (size 1.27 1.27)) (justify left))
     )
-    (property "Value" "4K7" (id 1) (at 128.27 94.2339 0)
+    (property "Value" "4K7" (id 1) (at 132.08 95.25 0)
       (effects (font (size 1.27 1.27)) (justify left))
     )
-    (property "Footprint" "Resistor_THT:R_Array_SIP9" (id 2) (at 130.175 92.71 90)
+    (property "Footprint" "Resistor_THT:R_Array_SIP9" (id 2) (at 103.505 92.71 90)
       (effects (font (size 1.27 1.27)) hide)
     )
-    (property "Datasheet" "http://www.vishay.com/docs/31509/csc.pdf" (id 3) (at 118.11 92.71 0)
+    (property "Datasheet" "http://www.vishay.com/docs/31509/csc.pdf" (id 3) (at 115.57 92.71 0)
       (effects (font (size 1.27 1.27)) hide)
     )
@@
     (pin "1")
   )
-  (symbol (lib_id "power:+5V") (at 107.95 87.63 0) (unit 1)
+  (symbol (lib_id "power:+5V") (at 125.73 87.63 0) (mirror y) (unit 1)
     (in_bom yes) (on_board yes) (fields_autoplaced)
-    (property "Reference" "#PWR045" (id 0) (at 107.95 91.44 0)
+    (property "Reference" "#PWR045" (id 0) (at 125.73 91.44 0)
       (effects (font (size 1.27 1.27)) hide)
     )
-    (property "Value" "+5V" (id 1) (at 107.95 82.55 0))
-    (property "Footprint" "" (id 2) (at 107.95 87.63 0)
+    (property "Value" "+5V" (id 1) (at 125.73 82.55 0))
+    (property "Footprint" "" (id 2) (at 125.73 87.63 0)
       (effects (font (size 1.27 1.27)) hide)
     )
-    (property "Datasheet" "" (id 3) (at 107.95 87.63 0)
+    (property "Datasheet" "" (id 3) (at 125.73 87.63 0)
       (effects (font (size 1.27 1.27)) hide)
     )
