File: v1_02/VGA.kicad_sch (KiCad schematic)
At the start: 27 parts, among them J9 DB15_Female_HighDensity_Mount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

Commit message: v1_02: Updated symbols/footprints for KiCAD9; fix all ERC/DRC warnings
Parts:
- J9: symbol Connector:DB15_Female_HighDensity_MountingHoles -> Connector:DE15_Socket_HighDensity_MountingHoles
- L1, L2, L3, L4, L5, L6: footprint Inductor_SMD:L_1206_3216Metric_Pad1.42x1.75mm_HandSolder -> Inductor_SMD:L_1206_3216Metric_Pad1.22x1.90mm_HandSolder
Changed lines of the file:
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@@
 			)
 		)
-		(property "Footprint" "Inductor_SMD:L_1206_3216Metric_Pad1.42x1.75mm_HandSolder"
+		(property "Footprint" "Inductor_SMD:L_1206_3216Metric_Pad1.22x1.90mm_HandSolder"
 			(at 101.6 87.63 0)
 			(effects
@@
 			)
 		)
-		(property "Description" ""
+		(property "Description" "Resistor, small symbol"
 			(at 71.12 140.97 0)
 			(effects
@@
 			)
 		)
-		(property "Description" ""
+		(property "Description" "Resistor, small symbol"
 			(at 69.85 72.39 0)
 			(effects
@@
 			)
 		)
-		(property "Footprint" "Inductor_SMD:L_1206_3216Metric_Pad1.42x1.75mm_HandSolder"
+		(property "Footprint" "Inductor_SMD:L_1206_3216Metric_Pad1.22x1.90mm_HandSolder"
 			(at 88.9 63.5 0)
 			(effects
@@
 	)
 	(symbol
-		(lib_id "Connector:DB15_Female_HighDensity_MountingHoles")
+		(lib_id "Connector:DE15_Socket_HighDensity_MountingHoles")
 		(at 177.8 92.71 0)
 		(unit 1)
@@
 			)
 		)
-		(property "Description" ""
+		(property "Description" "15-pin D-SUB connector, socket (female), High density (3 columns), Triple Row, Generic, VGA-connector, Mounting Hole"
 			(at 177.8 92.71 0)
 			(effects
@@
 			)
 		)
-		(property "Description" ""
+		(property "Description" "Resistor, small symbol"
 			(at 71.12 151.13 0)
 			(effects
@@
 			)
 		)
-		(property "Description" ""
+		(property "Description" "Resistor, small symbol"
 			(at 69.85 96.52 0)
 			(effects
@@
 			)
 		)
-		(property "Description" ""
+		(property "Description" "Resistor, small symbol"
 			(at 114.3 63.5 0)
 			(effects
@@
 			)
 		)
-		(property "Description" ""
+		(property "Description" "Resistor, small symbol"
 			(at 76.2 63.5 0)
 			(effects
@@
 			)
 		)
-		(property "Description" ""
+		(property "Description" "Power symbol creates a global label with name \"GND\" , ground"
 			(at 166.37 107.95 0)
 			(effects
@@
 			)
 		)
-		(property "Footprint" "Inductor_SMD:L_1206_3216Metric_Pad1.42x1.75mm_HandSolder"
+		(property "Footprint" "Inductor_SMD:L_1206_3216Metric_Pad1.22x1.90mm_HandSolder"
 			(at 101.6 113.03 0)
 			(effects
@@
 			)
 		)
-		(property "Description" ""
+		(property "Description" "Resistor, small symbol"
 			(at 114.3 113.03 0)
 			(effects
@@
 			)
 		)
-		(property "Description" ""
+		(property "Description" "Resistor, small symbol"
 			(at 76.2 113.03 0)
 			(effects
@@
 			)
 		)
-		(property "Description" ""
+		(property "Description" "Power symbol creates a global label with name \"GND\" , ground"
 			(at 139.7 132.08 0)
 			(effects
@@
 			)
 		)
-		(property "Description" ""
+		(property "Description" "Resistor, small symbol"
 			(at 76.2 87.63 0)
 			(effects
@@
 			)
 		)
-		(property "Footprint" "Inductor_SMD:L_1206_3216Metric_Pad1.42x1.75mm_HandSolder"
+		(property "Footprint" "Inductor_SMD:L_1206_3216Metric_Pad1.22x1.90mm_HandSolder"
 			(at 88.9 87.63 0)
 			(effects
@@
 			)
 		)
-		(property "Description" ""
+		(property "Description" "Resistor, small symbol"
 			(at 69.85 121.92 0)
 			(effects
@@
 			)
 		)
-		(property "Footprint" "Inductor_SMD:L_1206_3216Metric_Pad1.42x1.75mm_HandSolder"
+		(property "Footprint" "Inductor_SMD:L_1206_3216Metric_Pad1.22x1.90mm_HandSolder"
 			(at 101.6 63.5 0)
 			(effects
@@
 			)
 		)
-		(property "Footprint" "Inductor_SMD:L_1206_3216Metric_Pad1.42x1.75mm_HandSolder"
+		(property "Footprint" "Inductor_SMD:L_1206_3216Metric_Pad1.22x1.90mm_HandSolder"
 			(at 88.9 113.03 0)
 			(effects
@@
 			)
 		)
-		(property "Description" ""
+		(property "Description" "Resistor, small symbol"
 			(at 114.3 87.63 0)
 			(effects
